Commit message: Mirror the real SO-101 live + Piper X arm from actuacore-feetech
Sync with today's actuacore-feetech commits, taking only what the world
editor needs:

- world/assets/so101: his latest URDF (calibrated camera mount, OpenCV
  camera frame, new colours). STLs/calibration were already identical.
- world/assets/piper: Piper X arm description (URDF + OBJ visuals + MTL
  colours; collision STLs skipped — the loader ignores collision geometry).
- urdf-loader: .obj mesh support (merged sub-meshes, flat normals), MTL Kd
  colour backfill when the URDF declares no material, and <mimic> joints
  (the Piper's right finger tracks the left; its slider is hidden).
- Live mirroring: tools/so101_ws_bridge.py runs on the viewer laptop and
  forwards the handler's msgpack ZMQ state stream (tcp port derived from
  the same blake2b channel hash as actuacore's runtime_paths) to
  ws://localhost:8765 as JSON; world/lib/live-drive.js subscribes with
  auto-reconnect (plus a msgpack fallback decoder) and drives every placed
  arm whose joint names match. Live panel in the shelf shows status/Hz;
  per-instance "live" checkbox hand-poses one arm while others mirror.
- launch.json: autoPort so a second session's dev server can coexist.

Robot side needs ACTUACORE_ZMQ_TRANSPORT=tcp on the handler (channel
so101_r) — see README.

Co-Authored-By: Claude Opus 5 <noreply@anthropic.com>

File: world/assets/so101/so101_new_calib.urdf (robot description, URDF)
Before this commit: robot so101_new_calib, 10 links, 9 joints
Joints:
- joint camera_joint: origin xyz=0 0 0.015 rpy=0 0 0 -> xyz=0 0 0.015 rpy=-1.5708 0 0
- joint camera_mount_base_joint: origin xyz=0.0077 0.0001 -0.0234 rpy=-1.5708 0 0 -> xyz=0.0077 0.0203 -0.0234 rpy=-1.5708 0 0

Commit message: Pull Theo's 20-degree camera tilt into the SO-101 URDF
actuacore 5a9f466 "tilt camera" changes one line — camera_joint rpy -1.5708 ->
-1.9199, i.e. 0.3491 rad of downward tilt on the optical frame. Our copy predated
it, so the world was rendering the untilted lens.

Nothing in the conversion changes: the three.js camera still looks along
camera_link's +z, which is what the frame means. Measured after the update, the
view direction and that axis are 0.00 degrees apart, and the lens now sits 20.0
degrees off the gripper approach — Theo's tilt, arriving by copying a file.

Reworded the comment to say so, because that is the property worth keeping: the
aim belongs to the URDF, the code only flips -z to +z.

Co-Authored-By: Claude Opus 5 <noreply@anthropic.com>

File: world/assets/so101/so101_new_calib.urdf (robot description, URDF)
Before this commit: robot so101_new_calib, 10 links, 9 joints
Joints:
- joint camera_joint: origin xyz=0 0 0.015 rpy=-1.5708 0 0 -> xyz=0 0 0.015 rpy=-1.9199 0 0
